Commit message: 修复文件路径

File: src/openarm_moveit_config/config/mujoco_openarm_bimanual_cam.urdf (robot description, URDF)
Before this commit: robot openarm, 29 links, 28 joints
Links:
- link camera_link: geometry collision box size=0.02505 0.09 0.025; visual mesh filename=file:///home/yuxia/work_ws/install/openarm_description/shar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
