Commit message: 修改苹果URDF配置，并更新MoveIt相关启动文件，新增苹果模型文件夹

File: src/openarm_description_team/urdf/apple.urdf (robot description, URDF)
Before this commit: robot apple, 1 links, 1 joints
Links:
- link apple_link: geometry collision sphere radius=0.04; visual mesh filename=package://openarm_description_team/urdf/Red_Apple_model_526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 scale=0.01 0.01 0.01
